File: SigmaLink-USBi.kicad_pcb (KiCad board)
At the start: 2 copper layers, 64 x 39 mm, 31 parts, among them J1 USB_B, J2 Program, J3 Target, U1 LM1117-3.3, U2 24LC512, U3 CY7C68013A-56, U4 MAX809, U5 74LVC2G66, U6 TPS2051B, Y1 24MHz

Commit message: refactoring, move to 8.0
Parts:
- removed RN1: 510, Resistor_SMD:R_Array_Convex_4x0603
- removed RN2, RN4: 4.7k, Resistor_SMD:R_Array_Convex_4x0603
- removed RN3: 10k, Resistor_SMD:R_Array_Convex_4x0603
- added C10: 10V 47uF X5R, Capacitor_SMD:C_1206_3216Metric, F.Cu at (142.1, 94.4)
- added C12: 100n, Capacitor_SMD:C_0402_1005Metric, F.Cu at (161.6, 107.9)
- added C8: 10V 47uF X5R, Capacitor_SMD:C_1206_3216Metric, F.Cu at (131.7, 113.7)
- added R1: 4k7, Resistor_SMD:R_0402_1005Metric, F.Cu at (157.0, 89.8)
- added R10: 10k, Resistor_SMD:R_0402_1005Metric, F.Cu at (167.2, 108.6)
- added R11: 510, Resistor_SMD:R_0402_1005Metric, F.Cu at (149.0, 109.9)
- added R12: 510, Resistor_SMD:R_0402_1005Metric, F.Cu at (148.0, 109.9)
- added R13: 510, Resistor_SMD:R_0402_1005Metric, F.Cu at (150.0, 109.9)
- added R14: 510, Resistor_SMD:R_0402_1005Metric, F.Cu at (142.4, 109.7)
- added R2: 4k7, Resistor_SMD:R_0402_1005Metric, F.Cu at (162.4, 100.3)
- added R3: 4k7, Resistor_SMD:R_0402_1005Metric, F.Cu at (162.4, 101.3)
- added R4: 4k7, Resistor_SMD:R_0402_1005Metric, F.Cu at (162.4, 102.5)
- added R5: 10k, Resistor_SMD:R_0402_1005Metric, F.Cu at (157.1, 97.2)
- added R8: 4k7, Resistor_SMD:R_0402_1005Metric, F.Cu at (150.4, 107.1)
- added R9: 4k7, Resistor_SMD:R_0402_1005Metric, F.Cu at (152.8, 102.4)
- C1: value 100µ -> 10V 47uF X5R; footprint Capacitor_SMD:CP_Elec_6.3x5.3 -> Capacitor_SMD:C_1206_3216Metric
- C11, C13, C5, C6, C7, C9: footprint Capacitor_SMD:C_0603_1608Metric_Pad1.05x0.95mm_HandSolder -> Capacitor_SMD:C_0402_1005Metric
- C2: value 220µ -> 100n; footprint Capacitor_SMD:CP_Elec_6.3x5.3 -> Capacitor_SMD:C_0402_1005Metric
- D4: value B5819W -> B5819W SL
- R6: footprint Resistor_SMD:R_0603_1608Metric_Pad1.05x0.95mm_HandSolder -> Resistor_SMD:R_0402_1005Metric
- R7: value 4.7k -> 10k; footprint Resistor_SMD:R_0603_1608Metric_Pad1.05x0.95mm_HandSolder -> Resistor_SMD:R_0402_1005Metric
- U1: value LM1117-3.3 -> AMS1117-3.3
- Y1: footprint Crystal:Crystal_HC49-4H_Vertical -> Crystal:Crystal_SMD_5032-2Pin_5.0x3.2mm
- moved D4 12.4 mm to (152.2, 108.5)
- moved C11 10.9 mm to (162.5, 103.9), turned to 0 degrees
- moved C13 10.8 mm to (164.7, 111.4), turned to 90 degrees
- moved C4 8.15 mm to (139.3, 86.0), turned to 90 degrees
- moved U6 7.44 mm to (167.2, 111.0)
- moved C2 7.42 mm to (144.5, 93.4)
- moved R7 7.04 mm to (164.0, 90.7)
- moved C7 6.20 mm to (146.7, 88.6)
- moved Y1 4.07 mm to (141.1, 89.8)
- moved C3 3.18 mm to (141.1, 86.0), turned to 90 degrees
- moved C5 3.07 mm to (155.1, 90.3), turned to -90 degrees
- moved C9 1.91 mm to (155.1, 96.2), turned to -90 degrees
- moved C6 1.42 mm to (144.9, 89.8)
- moved C1 1.27 mm to (129.2, 113.7)
- moved U4 0.89 mm to (159.9, 89.2)
Connections:
- net /~TLATCH2 renamed /~{TLATCH2}
- net /~TLATCH3 renamed /~{TLATCH3}
- net /~TLATCH4 renamed /~{TLATCH4}
- net /~TLATCH5 renamed /~{TLATCH5}
- net Net-(C11-Pad1) renamed /Vcc(prom)
- J3 pad 11: /~TLATCH1 -> /~{TLATCH1}
- R7 pad 1: Net-(R7-Pad1) -> /~{TLATCH1}
- R7 pad 2: Net-(R7-Pad2) -> +3V3
- U3 pad 1: (no net) -> unconnected-(U3-RDY0/SLRD-Pad1)
- U3 pad 13: (no net) -> unconnected-(U3-IFCLK-Pad13)
- U3 pad 2: (no net) -> unconnected-(U3-RDY1/SLWR-Pad2)
- U3 pad 23: (no net) -> unconnected-(U3-PB5/FD5-Pad23)
- U3 pad 24: (no net) -> unconnected-(U3-PB6/FD6-Pad24)
- U3 pad 25: (no net) -> unconnected-(U3-PB7/FD7-Pad25)
- U3 pad 29: (no net) -> unconnected-(U3-CTL0/FLAGA-Pad29)
- U3 pad 30: (no net) -> unconnected-(U3-CTL1/FLAGB-Pad30)
- U3 pad 31: (no net) -> unconnected-(U3-CTL2/FLAGC-Pad31)
- U3 pad 35: /~TLATCH1 -> /~{TLATCH1}
- U3 pad 42: Net-(R7-Pad2) -> Net-(U3-~{RESET})
- U3 pad 44: (no net) -> unconnected-(U3-WAKEUP-Pad44)
- U3 pad 45: (no net) -> unconnected-(U3-PD0/FD8-Pad45)
- U3 pad 46: (no net) -> unconnected-(U3-PD1/FD9-Pad46)
- U3 pad 47: (no net) -> unconnected-(U3-PD2/FD10-Pad47)
- U3 pad 48: (no net) -> unconnected-(U3-PD3/FD11-Pad48)
- U3 pad 49: (no net) -> unconnected-(U3-PD4/FD12-Pad49)
- U3 pad 50: (no net) -> unconnected-(U3-PD5/FD13-Pad50)
- U3 pad 51: (no net) -> unconnected-(U3-PD6/FD14-Pad51)
- U3 pad 52: (no net) -> unconnected-(U3-PD7/FD15-Pad52)
- U4 pad 2: Net-(R7-Pad1) -> Net-(U4-~{RESET})
- U6 pad 3: (no net) -> unconnected-(U6-~{OC}-Pad3)
Routing:
- net /~{TLATCH1}: track 0.00 -> 46.9 mm, vias 0 -> 2
- net /~TLATCH1: track 33.9 -> 0.00 mm, vias 3 -> 0
- net +3V3: track 115.7 -> 91.6 mm, vias 11 -> 17
- net /USB_EN: track 48.2 -> 31.9 mm, vias 4 -> 3
- net /Vcc(prom): track 30.0 -> 18.5 mm, vias 3 -> 0
- net /TVCC: track 32.7 -> 21.7 mm
- net /XTALO: track 17.8 -> 7.84 mm
- net /XTALI: track 19.3 -> 10.9 mm
- net GND: track 5.53 -> 0.04 mm, vias 516 -> 269
- net Net-(D2-K2): track 12.9 -> 7.57 mm
- net /TSCL: track 27.5 -> 22.5 mm, vias 2 -> 0
- net Net-(J2-G1): track 9.88 -> 5.30 mm, vias 1 -> 0
- net /SDA: track 26.9 -> 22.6 mm, vias 3 -> 2
- net Net-(D2-K1): track 5.88 -> 1.65 mm
- net /TSDA: track 22.1 -> 18.0 mm, vias 2 -> 0
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- added copper zone on B.Cu, net +3V3
Other:
- net class Default removed
- net class Power removed

Commit message: gerbers
Parts:
- removed U3: CY7C68013A-56, Package_DFN_QFN:QFN-56-1EP_8x8mm_P0.5mm_EP4.6x5.3mm
- added U7: CY7C68013A-56LTX, Package_DFN_QFN:QFN-56-1EP_8x8mm_P0.5mm_EP4.5x5.2mm_ThermalVias_TopTented, F.Cu at (150.0, 93.7)
- C3, C4: footprint Capacitor_SMD:C_0603_1608Metric_Pad1.05x0.95mm_HandSolder -> Capacitor_SMD:C_0603_1608Metric
- moved F1 2.77 mm to (123.9, 111.4), turned to 180 degrees
- moved C2 0.21 mm to (144.3, 93.4)
- moved C7 0.17 mm to (146.7, 88.4)
- moved C5 0.12 mm to (155.2, 90.3)
- moved C6 0.12 mm to (144.8, 89.8)
- moved R7 0.10 mm to (164.0, 90.8)
Connections:
- net +3V3 renamed VCC
- R1 pad 2: Net-(U3-~{RESET}) -> /RESET
Routing:
- net +5V: track 52.6 -> 48.7 mm
- net Net-(J1-VBUS): track 14.3 -> 17.9 mm
- net Net-(U3-~{RESET}): track 2.89 -> 0.00 mm
- net /RESET: track 0.00 -> 2.89 mm
- net GND: vias 269 -> 254

Commit message: ordered
Parts:
- J2: footprint Connector_PinHeader_1.27mm:PinHeader_1x02_P1.27mm_Vertical -> Connector_PinHeader_2.54mm:PinHeader_1x02_P2.54mm_Vertical
- moved J2 0.91 mm to (151.0, 104.4)
- moved D4 0.70 mm to (152.9, 108.7)
Routing:
- net /LED_I2C: track 13.2 -> 14.4 mm
- net /LED_GPIO: track 13.5 -> 14.5 mm
- net /LED_SPI: track 14.0 -> 14.9 mm
- net /Vcc(prom): track 18.5 -> 19.2 mm
- net /SCL: track 24.2 -> 24.8 mm
- net GND: vias 254 -> 252
Other:
- outline, holes or cut-outs redrawn
- board text added: "SigmaLink USBi"
- board text removed: "SigmaLink USBi © 2019 Max Chan"
