File: SigmaLink-USBi.kicad_sch (KiCad schematic)
At the start: 42 parts, among them J1 USB_B, J2 Program, J3 Target, U1 AMS1117-3.3, U2 24LC512, U3 CY7C68013A-56, U4 MAX809, U5 74LVC2G66, U6 TPS2051B, Y1 24MHz

Commit message: gerbers
Parts:
- added U7: CY7C68013A-56LTX, Package_DFN_QFN:QFN-56-1EP_8x8mm_P0.5mm_EP4.5x5.2mm_ThermalVias_TopTented, symbol MCU_Cypress:CY7C68013A-56LTX
- C3, C4: footprint Capacitor_SMD:C_0603_1608Metric_Pad1.05x0.95mm_HandSolder -> Capacitor_SMD:C_0603_1608Metric
- U1: now in the parts list
- U3: now not fitted
Connections:
- net D+: now also U7.8 (D+)
- net D-: now also U7.9 (D-)
- net GND: now also U7.10 (AGND), U7.12 (GND), U7.14 (RESERVED), U7.26 (GND), U7.28 (GND), U7.41 (GND), U7.53 (GND), U7.56 (GND), U7.57 (EP), U7.6 (AGND)
- net LED_GPIO: now also U7.20 (PB2/FD2)
- net LED_I2C: now also U7.19 (PB1/FD1)
- net LED_SPI: now also U7.21 (PB3/FD3)
- net MCK: now also U7.54 (CLKOUT)
- net SCL: now also U7.15 (SCL)
- net SDA: now also U7.16 (SDA)
- net TCLK: now also U7.40 (PA7/FLAGD/~{SLCS})
- net TDATA: now also U7.33 (PA0/~{INT0})
- net TOUT: now also U7.34 (PA1/~{INT1})
- net TRESET: now also U7.18 (PB0/FD0)
- net USB_EN: now also U7.22 (PB4/FD4)
- net XTALI: now also U7.5 (XTALIN)
- net XTALO: now also U7.4 (XTALOUT)
- net ~{TLATCH1}: now also U7.35 (PA2/SLOE)
- net ~{TLATCH2}: now also U7.36 (PA3/WU2)
- net ~{TLATCH3}: now also U7.37 (PA4/FIOADDR0)
- net ~{TLATCH4}: now also U7.38 (PA5/FIOADDR1)
- net ~{TLATCH5}: now also U7.39 (PA6/PKTEND)
- net RESET: now reaches R1.2, U3.42 (~{RESET})
- net RESET: now also U7.42 (~{RESET})
- net +3V3 renamed VCC
- net VCC: now also U7.11 (VCC), U7.17 (VCC), U7.27 (VCC), U7.3 (AVCC), U7.32 (VCC), U7.43 (VCC), U7.55 (VCC), U7.7 (AVCC)
- no-connect marks 19 -> 37

Commit message: ordered
Parts:
- J2: footprint Connector_PinHeader_1.27mm:PinHeader_1x02_P1.27mm_Vertical -> Connector_PinHeader_2.54mm:PinHeader_1x02_P2.54mm_Vertical
Changed lines of the file:
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@@
 			)
 		)
-		(property "Footprint" "Connector_PinHeader_1.27mm:PinHeader_1x02_P1.27mm_Vertical"
+		(property "Footprint" "Connector_PinHeader_2.54mm:PinHeader_1x02_P2.54mm_Vertical"
 			(at 135.2804 91.44 90)
 			(effects
